File: PCB/PCB.kicad_pcb (KiCad board)
At the start: 4 copper layers, 0 parts

Commit message: PCB ready for layout
Parts:
- added C1: 10u, Capacitor_SMD:C_0402_1005Metric_Pad0.74x0.62mm_HandSolder, F.Cu at (143.3, 111.8)
- added C3: 0.1u, Capacitor_SMD:C_0402_1005Metric_Pad0.74x0.62mm_HandSolder, F.Cu at (143.3, 113.8)
- added P1: SEN-11574, footprints:Heart_headers, F.Cu at (158.6, 110.0)
- added R1: 100k, Resistor_SMD:R_0402_1005Metric_Pad0.72x0.64mm_HandSolder, F.Cu at (163.1, 73.9)
- added R2: 220, Resistor_SMD:R_0402_1005Metric_Pad0.72x0.64mm_HandSolder, F.Cu at (163.1, 75.9)
- added R3: 1k, Resistor_SMD:R_0402_1005Metric_Pad0.72x0.64mm_HandSolder, F.Cu at (163.1, 77.9)
- added R4: 220, Resistor_SMD:R_0402_1005Metric_Pad0.72x0.64mm_HandSolder, F.Cu at (163.1, 79.9)
- added R5: 220, Resistor_SMD:R_0402_1005Metric_Pad0.72x0.64mm_HandSolder, F.Cu at (163.1, 81.9)
- added R6: 220, Resistor_SMD:R_0402_1005Metric_Pad0.72x0.64mm_HandSolder, F.Cu at (163.1, 83.9)
- added R7: 220, Resistor_SMD:R_0402_1005Metric_Pad0.72x0.64mm_HandSolder, F.Cu at (163.1, 85.8)
- added R8: 220, Resistor_SMD:R_0402_1005Metric_Pad0.72x0.64mm_HandSolder, F.Cu at (163.1, 87.8)
- added U1: TinyS3_Symbol, footprints:TinyS3D_headers, F.Cu at (132.2, 96.4)
- added U2: ADXL345, footprints:ADXL345_header, F.Cu at (146.8, 84.5)
- added U3: ST7789V, footprints:LCD_header, F.Cu at (153.7, 99.9)
- added U4: switch3, footprints:Buttons_header, F.Cu at (148.6, 107.0)

Commit message: Added USBC measurement to footprint
Parts:
- removed C1: 10u, Capacitor_SMD:C_0402_1005Metric_Pad0.74x0.62mm_HandSolder
- removed C3: 0.1u, Capacitor_SMD:C_0402_1005Metric_Pad0.74x0.62mm_HandSolder
- removed P1: SEN-11574, footprints:Heart_headers
- removed R1: 100k, Resistor_SMD:R_0402_1005Metric_Pad0.72x0.64mm_HandSolder
- removed R2, R4, R5, R6, R7, R8: 220, Resistor_SMD:R_0402_1005Metric_Pad0.72x0.64mm_HandSolder
- removed R3: 1k, Resistor_SMD:R_0402_1005Metric_Pad0.72x0.64mm_HandSolder
- removed U1: TinyS3_Symbol, footprints:TinyS3D_headers
- removed U2: ADXL345, footprints:ADXL345_header
- removed U3: ST7789V, footprints:LCD_header
- removed U4: switch3, footprints:Buttons_header

Commit message: Floorplan, routing WIP
Parts:
- added C1: 10u, Capacitor_SMD:C_0402_1005Metric_Pad0.74x0.62mm_HandSolder, F.Cu at (123.4, 104.6)
- added C3: 0.1u, Capacitor_SMD:C_0402_1005Metric_Pad0.74x0.62mm_HandSolder, F.Cu at (123.4, 99.9)
- added P1: SEN-11574, footprints:Heart_headers, F.Cu at (115.0, 96.8)
- added R1: 100k, Resistor_SMD:R_0402_1005Metric_Pad0.72x0.64mm_HandSolder, F.Cu at (120.6, 86.7)
- added R2: 220, Resistor_SMD:R_0402_1005Metric_Pad0.72x0.64mm_HandSolder, F.Cu at (123.5, 86.7)
- added R3: 1k, Resistor_SMD:R_0402_1005Metric_Pad0.72x0.64mm_HandSolder, F.Cu at (121.1, 99.3)
- added R4: 220, Resistor_SMD:R_0402_1005Metric_Pad0.72x0.64mm_HandSolder, F.Cu at (145.2, 109.6)
- added R5: 220, Resistor_SMD:R_0402_1005Metric_Pad0.72x0.64mm_HandSolder, F.Cu at (145.2, 104.5)
- added R6: 220, Resistor_SMD:R_0402_1005Metric_Pad0.72x0.64mm_HandSolder, F.Cu at (145.2, 101.9)
- added R7: 220, Resistor_SMD:R_0402_1005Metric_Pad0.72x0.64mm_HandSolder, F.Cu at (123.5, 89.3)
- added R8: 220, Resistor_SMD:R_0402_1005Metric_Pad0.72x0.64mm_HandSolder, F.Cu at (123.5, 91.8)
- added U1: TinyS3_Symbol, footprints:TinyS3D_headers, F.Cu at (134.3, 96.9)
- added U2: ADXL345, footprints:ADXL345_header, F.Cu at (151.1, 87.3)
- added U3: ST7789V, footprints:LCD_header, F.Cu at (134.1, 67.0)
- added U4: switch3, footprints:Buttons_header, F.Cu at (117.1, 113.9)
Other:
- board outline added: 56 x 55 mm
